Commit message: feat: prepare EVRENOS real vehicle stack for safe hardware integration
* harden STM32 bridge with motion enable interlock
* add linear and angular velocity clamps
* reject NaN/Inf cmd_vel inputs and command zero
* add startup/reconnect zero interlock and watchdog protection
* preserve safe shutdown with redundant zero frames
* add runtime disable-only motion safety latch
* expose safety parameters through real base, mapping, and Nav2 launches
* add Unitree L1 TF chain: base_link -> lidar_link -> unilidar_lidar
* align Unitree PointCloud2 frame with unilidar_lidar
* keep pointcloud_to_laserscan target frame on lidar_link
* add optional BNO055 driver integration and configuration
* connect BNO055 /imu/data to EKF with explicit covariances
* preserve existing SLAM, Nav2, and EKF tuning
* fix LiDAR launch argument forwarding in real mapping launch
* add real vehicle operations and preflight runbook
* add safe mapping, localization, map save, low-speed test, and emergency-stop procedures
* validate TF ownership and remove duplicate/conflicting frame publishers
* verify hardwareless startup with STM32, LiDAR, and BNO055 disabled
* confirm clean build, launch, shutdown, and ROS graph behavior

Validated with:

* python3 -m py_compile
* git diff --check
* xacro + check_urdf
* colcon build
* hardwareless ROS 2 launch and TF/topic inspection

File: src/yektemak_description/urdf/evrenos_sensors.xacro (robot description, xacro)
@@ -23,10 +23,22 @@
   </link>
   <joint name="lidar_joint" type="fixed">
-    <parent link="body_link"/>
+    <parent link="base_link"/>
     <child link="lidar_link"/>
-    <!-- Upper/front portion of vehicle -->
+    <!--
+      Preserve the original mount pose relative to base_link.
+      The previous body_link parent contributes
+      base_height / 2.0 + 0.08 in Z.
+    -->
     <origin
-      xyz="0.12 0 0.31"
+      xyz="0.12 0 ${base_height / 2.0 + 0.08 + 0.31}"
       rpy="0 0 0"/>
+  </joint>
+  <!-- Unitree L1 PointCloud2 measurement/output frame -->
+  <link name="unilidar_lidar"/>
+  <joint name="unilidar_lidar_joint" type="fixed">
+    <parent link="lidar_link"/>
+    <child link="unilidar_lidar"/>
+    <!-- Replace only if a verified sensor-to-mount transform is measured. -->
+    <origin xyz="0 0 0" rpy="0 0 0"/>
   </joint>
   <!-- ====================================================== -->

Commit message: feat: finalize EVRENOS real vehicle LiDAR and IMU integration
* integrate Unitree L1 built-in IMU into the real vehicle stack
* route Unitree IMU output to the existing /imu/data EKF input
* add unilidar_imu frame to the EVRENOS robot TF tree
* add official Unitree L1 lidar-to-IMU fixed transform
* propagate IMU topic and frame parameters through sensor, mapping and Nav2 launches
* keep BNO055 support optional and disabled by default
* prevent Unitree L1 and BNO055 from publishing /imu/data simultaneously
* preserve existing EKF fusion configuration and LiDAR point-cloud pipeline
* preserve STM32 safety, SLAM and Nav2 tuning
* ignore vendor Unitree ROS packages during colcon package discovery
* validate complete TF chain and hardware-disabled launch behavior
* verify full EVRENOS workspace build successfully

Final sensor architecture:
base_link -> lidar_link -> unilidar_lidar -> unilidar_imu

Unitree L1:

* point cloud frame: unilidar_lidar
* IMU topic: /imu/data
* IMU frame: unilidar_imu

Validation:

* git diff --check passed
* full colcon build passed (5 packages)
* hardwareless mapping launch passed
* dual-IMU conflict protection passed
* x86_64 and aarch64 Unitree SDK libraries verified

File: src/yektemak_description/urdf/evrenos_sensors.xacro (robot description, xacro)
@@ -41,4 +41,12 @@
     <!-- Replace only if a verified sensor-to-mount transform is measured. -->
     <origin xyz="0 0 0" rpy="0 0 0"/>
+  </joint>
+  <!-- Unitree L1 built-in IMU measurement/output frame -->
+  <link name="unilidar_imu"/>
+  <joint name="unilidar_imu_joint" type="fixed">
+    <parent link="unilidar_lidar"/>
+    <child link="unilidar_imu"/>
+    <!-- Official Unitree L1 LiDAR-to-IMU transform. -->
+    <origin xyz="-0.007698 -0.014655 0.00667" rpy="0 0 0"/>
   </joint>
   <!-- ====================================================== -->
