Commit message: feat: tune EVRENOS SLAM and Nav2 simulation pipeline, stabilize EVRENOS SLAM timing and tune Nav2 simulation

File: src/yektemak_description/urdf/evrenos_base.xacro (robot description, xacro)
@@ -2,10 +2,11 @@
 <robot xmlns:xacro="http://www.ros.org/wiki/xacro">
   <!-- EVRENOS simplified physical chassis -->
-  <xacro:property name="base_length" value="1.05"/>
-  <xacro:property name="base_width"  value="0.78"/>
-  <xacro:property name="base_height" value="0.24"/>
-  <xacro:property name="base_ground_clearance" value="0.18"/>
+  <xacro:property name="vehicle_scale" value="0.80"/>
+  <xacro:property name="base_length" value="${1.05 * vehicle_scale}"/>
+  <xacro:property name="base_width"  value="${0.78 * vehicle_scale}"/>
+  <xacro:property name="base_height" value="${0.24 * vehicle_scale}"/>
+  <xacro:property name="base_ground_clearance" value="${0.18 * vehicle_scale}"/>
   <!-- 84 kg chassis + 4 x 4 kg wheel ~= 100 kg -->
-  <xacro:property name="base_mass" value="84.0"/>
+  <xacro:property name="base_mass" value="${84.0 * vehicle_scale ** 3}"/>
   <link name="base_footprint"/>
   <link name="base_link">

File: src/yektemak_description/urdf/evrenos_body.xacro (robot description, xacro)
@@ -14,7 +14,7 @@
     <!-- Center armored body -->
     <visual>
-      <origin xyz="-0.05 0 0.10" rpy="0 0 0"/>
+      <origin xyz="${-0.05 * vehicle_scale} 0 ${0.10 * vehicle_scale}" rpy="0 0 0"/>
       <geometry>
-        <box size="0.68 0.74 0.22"/>
+        <box size="${0.68 * vehicle_scale} ${0.74 * vehicle_scale} ${0.22 * vehicle_scale}"/>
       </geometry>
       <material name="evrenos_body"/>
@@ -22,7 +22,7 @@
     <!-- Front sloped armor -->
     <visual>
-      <origin xyz="0.34 0 0.055" rpy="0 -0.30 0"/>
+      <origin xyz="${0.34 * vehicle_scale} 0 ${0.055 * vehicle_scale}" rpy="0 -0.30 0"/>
       <geometry>
-        <box size="0.42 0.74 0.17"/>
+        <box size="${0.42 * vehicle_scale} ${0.74 * vehicle_scale} ${0.17 * vehicle_scale}"/>
       </geometry>
       <material name="evrenos_metal"/>
@@ -30,7 +30,7 @@
     <!-- Rear upper armor -->
     <visual>
-      <origin xyz="-0.39 0 0.06" rpy="0 0.20 0"/>
+      <origin xyz="${-0.39 * vehicle_scale} 0 ${0.06 * vehicle_scale}" rpy="0 0.20 0"/>
       <geometry>
-        <box size="0.30 0.72 0.17"/>
+        <box size="${0.30 * vehicle_scale} ${0.72 * vehicle_scale} ${0.17 * vehicle_scale}"/>
       </geometry>
       <material name="evrenos_body"/>
@@ -38,7 +38,7 @@
     <!-- Roof -->
     <visual>
-      <origin xyz="-0.05 0 0.235" rpy="0 0 0"/>
+      <origin xyz="${-0.05 * vehicle_scale} 0 ${0.235 * vehicle_scale}" rpy="0 0 0"/>
       <geometry>
-        <box size="0.54 0.58 0.06"/>
+        <box size="${0.54 * vehicle_scale} ${0.58 * vehicle_scale} ${0.06 * vehicle_scale}"/>
       </geometry>
       <material name="evrenos_dark"/>
@@ -46,7 +46,7 @@
     <!-- Front center armor panel -->
     <visual>
-      <origin xyz="0.50 0 0.015" rpy="0 -0.35 0"/>
+      <origin xyz="${0.50 * vehicle_scale} 0 ${0.015 * vehicle_scale}" rpy="0 -0.35 0"/>
       <geometry>
-        <box size="0.18 0.60 0.12"/>
+        <box size="${0.18 * vehicle_scale} ${0.60 * vehicle_scale} ${0.12 * vehicle_scale}"/>
       </geometry>
       <material name="evrenos_body"/>
@@ -54,7 +54,7 @@
     <!-- Front left lamp -->
     <visual>
-      <origin xyz="0.575 0.20 0.015" rpy="0 0 0"/>
+      <origin xyz="${0.575 * vehicle_scale} ${0.20 * vehicle_scale} ${0.015 * vehicle_scale}" rpy="0 0 0"/>
       <geometry>
-        <box size="0.035 0.11 0.07"/>
+        <box size="${0.035 * vehicle_scale} ${0.11 * vehicle_scale} ${0.07 * vehicle_scale}"/>
       </geometry>
       <material name="evrenos_light"/>
@@ -62,7 +62,7 @@
     <!-- Front center lamp -->
     <visual>
-      <origin xyz="0.575 0 0.015" rpy="0 0 0"/>
+      <origin xyz="${0.575 * vehicle_scale} 0 ${0.015 * vehicle_scale}" rpy="0 0 0"/>
       <geometry>
-        <box size="0.035 0.11 0.07"/>
+        <box size="${0.035 * vehicle_scale} ${0.11 * vehicle_scale} ${0.07 * vehicle_scale}"/>
       </geometry>
       <material name="evrenos_light"/>
@@ -70,7 +70,7 @@
     <!-- Front right lamp -->
     <visual>
-      <origin xyz="0.575 -0.20 0.015" rpy="0 0 0"/>
+      <origin xyz="${0.575 * vehicle_scale} ${-0.20 * vehicle_scale} ${0.015 * vehicle_scale}" rpy="0 0 0"/>
       <geometry>
-        <box size="0.035 0.11 0.07"/>
+        <box size="${0.035 * vehicle_scale} ${0.11 * vehicle_scale} ${0.07 * vehicle_scale}"/>
       </geometry>
       <material name="evrenos_light"/>
@@ -85,5 +85,5 @@
     <child link="body_link"/>
     <origin
-      xyz="0 0 ${base_height / 2.0 + 0.08}"
+      xyz="0 0 ${base_height / 2.0 + 0.08 * vehicle_scale}"
       rpy="0 0 0"/>
   </joint>

File: src/yektemak_description/urdf/evrenos_gazebo.xacro (robot description, xacro)
@@ -70,9 +70,9 @@
       <right_joint>rear_right_wheel_joint</right_joint>
       <!-- Front wheel pair -->
-      <wheel_separation>1.065</wheel_separation>
-      <wheel_diameter>0.45</wheel_diameter>
+      <wheel_separation>${track_width}</wheel_separation>
+      <wheel_diameter>${2.0 * wheel_radius}</wheel_diameter>
       <!-- Rear wheel pair -->
-      <wheel_separation>1.065</wheel_separation>
-      <wheel_diameter>0.45</wheel_diameter>
+      <wheel_separation>${track_width}</wheel_separation>
+      <wheel_diameter>${2.0 * wheel_radius}</wheel_diameter>
       <max_wheel_torque>120.0</max_wheel_torque>
       <max_wheel_acceleration>2.0</max_wheel_acceleration>

File: src/yektemak_description/urdf/evrenos_sensors.xacro (robot description, xacro)
@@ -31,5 +31,5 @@
     -->
     <origin
-      xyz="0.12 0 ${base_height / 2.0 + 0.08 + 0.31}"
+      xyz="${0.12 * vehicle_scale} 0 ${base_height / 2.0 + (0.08 + 0.31) * vehicle_scale}"
       rpy="0 0 0"/>
   </joint>
@@ -67,5 +67,5 @@
     <!-- Front facing camera -->
     <origin
-      xyz="0.48 0 0.14"
+      xyz="${0.48 * vehicle_scale} 0 ${0.14 * vehicle_scale}"
       rpy="0 0 0"/>
   </joint>
@@ -96,5 +96,5 @@
     <!-- Close to vehicle center / center of mass -->
     <origin
-      xyz="0 0 0.05"
+      xyz="0 0 ${0.05 * vehicle_scale}"
       rpy="0 0 0"/>
   </joint>
@@ -116,5 +116,5 @@
     <!-- Upper rear section -->
     <origin
-      xyz="-0.24 0 0.32"
+      xyz="${-0.24 * vehicle_scale} 0 ${0.32 * vehicle_scale}"
       rpy="0 0 0"/>
   </joint>

File: src/yektemak_description/urdf/evrenos_wheels.xacro (robot description, xacro)
@@ -2,7 +2,7 @@
 <robot xmlns:xacro="http://www.ros.org/wiki/xacro">
   <!-- KTR wheel dimensions -->
-  <xacro:property name="wheel_radius" value="0.225"/>
-  <xacro:property name="wheel_width"  value="0.13"/>
-  <xacro:property name="wheel_mass"   value="4.0"/>
+  <xacro:property name="wheel_radius" value="${0.225 * vehicle_scale}"/>
+  <xacro:property name="wheel_width"  value="${0.13 * vehicle_scale}"/>
+  <xacro:property name="wheel_mass"   value="${4.0 * vehicle_scale ** 3}"/>
   <!--
     Temporary geometry derived from overall vehicle dimensions.
@@ -11,5 +11,5 @@
     wheelbase ~= 1.39 - 0.45 = 0.94 m
   -->
-  <xacro:property name="wheelbase" value="0.94"/>
+  <xacro:property name="wheelbase" value="${0.94 * vehicle_scale}"/>
   <!--
     Overall width = 1.195 m
@@ -18,5 +18,5 @@
       1.195 - 0.13 = 1.065 m
   -->
-  <xacro:property name="track_width" value="1.065"/>
+  <xacro:property name="track_width" value="${1.065 * vehicle_scale}"/>
   <xacro:property
     name="wheel_x_position"

Commit message: fix

File: src/yektemak_description/urdf/evrenos_base.xacro (robot description, xacro)
@@ -2,5 +2,5 @@
 <robot xmlns:xacro="http://www.ros.org/wiki/xacro">
   <!-- EVRENOS simplified physical chassis -->
-  <xacro:property name="vehicle_scale" value="0.80"/>
+  <xacro:property name="vehicle_scale" value="1.00"/>
   <xacro:property name="base_length" value="${1.05 * vehicle_scale}"/>
   <xacro:property name="base_width"  value="${0.78 * vehicle_scale}"/>

File: src/yektemak_description/urdf/evrenos_gazebo.xacro (robot description, xacro)
@@ -14,5 +14,5 @@
     <material>Gazebo/Black</material>
     <mu1>1.0</mu1>
-    <mu2>0.15</mu2>
+    <mu2>0.50</mu2>
     <fdir1>1 0 0</fdir1>
     <kp>1000000.0</kp>
@@ -24,5 +24,5 @@
     <material>Gazebo/Black</material>
     <mu1>1.0</mu1>
-    <mu2>0.15</mu2>
+    <mu2>0.50</mu2>
     <fdir1>1 0 0</fdir1>
     <kp>1000000.0</kp>
@@ -34,5 +34,5 @@
     <material>Gazebo/Black</material>
     <mu1>1.0</mu1>
-    <mu2>0.15</mu2>
+    <mu2>0.50</mu2>
     <fdir1>1 0 0</fdir1>
     <kp>1000000.0</kp>
@@ -44,5 +44,5 @@
     <material>Gazebo/Black</material>
     <mu1>1.0</mu1>
-    <mu2>0.15</mu2>
+    <mu2>0.50</mu2>
     <fdir1>1 0 0</fdir1>
     <kp>1000000.0</kp>
@@ -77,5 +77,5 @@
       <max_wheel_torque>120.0</max_wheel_torque>
       <max_wheel_acceleration>2.0</max_wheel_acceleration>
-      <update_rate>8.0</update_rate>
+      <update_rate>20.0</update_rate>
       <!-- Encoder-like wheel odometry -->
       <odometry_source>0</odometry_source>

File: src/yektemak_description/urdf/evrenos_sensors.xacro (robot description, xacro)
@@ -25,11 +25,7 @@
     <parent link="base_link"/>
     <child link="lidar_link"/>
-    <!--
-      Preserve the original mount pose relative to base_link.
-      The previous body_link parent contributes
-      base_height / 2.0 + 0.08 in Z.
-    -->
+    <!-- Front-facing mount; lidar_link center is 0.60 m above ground. -->
     <origin
-      xyz="${0.12 * vehicle_scale} 0 ${base_height / 2.0 + (0.08 + 0.31) * vehicle_scale}"
+      xyz="${base_length / 2.0 - 0.08} 0 ${0.60 - (base_ground_clearance + base_height / 2.0)}"
       rpy="0 0 0"/>
   </joint>
