Commit message: Improve pallet lifting geometry and contact friction

File: src/yektemak_description/urdf/yektemak_base.xacro (robot description, xacro)
@@ -2,11 +2,11 @@
 <robot xmlns:xacro="http://www.ros.org/wiki/xacro">
   <!-- Temel gövde ölçüleri metre cinsindedir. -->
-  <xacro:property name="base_length" value="1.20"/>
-  <xacro:property name="base_width" value="0.80"/>
-  <xacro:property name="base_height" value="0.25"/>
+  <xacro:property name="base_length" value="0.80"/>
+  <xacro:property name="base_width" value="0.38"/>
+  <xacro:property name="base_height" value="0.10"/>
   <!-- Gövdenin yerden yüksekliği -->
-  <xacro:property name="base_ground_clearance" value="0.15"/>
+  <xacro:property name="base_ground_clearance" value="0.04"/>
   <!-- Yaklaşık gövde kütlesi -->
-  <xacro:property name="base_mass" value="45.0"/>
+  <xacro:property name="base_mass" value="35.0"/>
   <!-- Zemindeki referans noktası -->
   <link name="base_footprint"/>

File: src/yektemak_description/urdf/yektemak_gazebo.xacro (robot description, xacro)
@@ -33,4 +33,10 @@
   <gazebo reference="lift_platform_link">
     <material>Gazebo/Yellow</material>
+    <mu1>10.0</mu1>
+    <mu2>10.0</mu2>
+    <kp>1000000.0</kp>
+    <kd>100.0</kd>
+    <minDepth>0.001</minDepth>
+    <maxVel>0.01</maxVel>
   </gazebo>
   <gazebo reference="front_marker_link">

File: src/yektemak_description/urdf/yektemak_lift.xacro (robot description, xacro)
@@ -2,10 +2,10 @@
 <robot xmlns:xacro="http://www.ros.org/wiki/xacro">
   <!-- Kaldırma platformu ölçüleri -->
-  <xacro:property name="lift_platform_length" value="0.90"/>
-  <xacro:property name="lift_platform_width" value="0.60"/>
-  <xacro:property name="lift_platform_height" value="0.05"/>
-  <xacro:property name="lift_platform_mass" value="8.0"/>
-  <xacro:property name="lift_platform_clearance" value="0.02"/>
-  <xacro:property name="lift_max_height" value="0.20"/>
+  <xacro:property name="lift_platform_length" value="0.68"/>
+  <xacro:property name="lift_platform_width" value="0.30"/>
+  <xacro:property name="lift_platform_height" value="0.04"/>
+  <xacro:property name="lift_platform_mass" value="6.0"/>
+  <xacro:property name="lift_platform_clearance" value="0.01"/>
+  <xacro:property name="lift_max_height" value="0.10"/>
   <!-- Paleti kaldıracak üst platform -->
   <link name="lift_platform_link">
@@ -60,5 +60,5 @@
       lower="0.0"
       upper="${lift_max_height}"
-      effort="2000.0"
+      effort="5000.0"
       velocity="0.10"/>
     <dynamics

File: src/yektemak_description/urdf/yektemak_markers.xacro (robot description, xacro)
@@ -1,7 +1,7 @@
 <robot xmlns:xacro="http://www.ros.org/wiki/xacro">
   <!-- Aracın +X yönündeki ön tarafını gösteren tampon -->
-  <xacro:property name="front_marker_length" value="0.05"/>
-  <xacro:property name="front_marker_width" value="0.50"/>
-  <xacro:property name="front_marker_height" value="0.10"/>
+  <xacro:property name="front_marker_length" value="0.04"/>
+  <xacro:property name="front_marker_width" value="0.28"/>
+  <xacro:property name="front_marker_height" value="0.06"/>
   <link name="front_marker_link">
     <visual>

File: src/yektemak_description/urdf/yektemak_ros2_control.xacro (robot description, xacro)
@@ -4,15 +4,19 @@
       <plugin>gazebo_ros2_control/GazeboSystem</plugin>
     </hardware>
-    <joint name="lift_platform_joint">
-      <command_interface name="position">
-        <param name="min">0.0</param>
-        <param name="max">0.20</param>
-      </command_interface>
-      <state_interface name="position">
-        <param name="initial_value">0.0</param>
-      </state_interface>
-      <state_interface name="velocity"/>
-      <state_interface name="effort"/>
-    </joint>
+  <joint name="lift_platform_joint">
+    <param name="pos_kp">6000.0</param>
+    <param name="pos_ki">50.0</param>
+    <param name="pos_kd">150.0</param>
+    <param name="pos_max_integral_error">100.0</param>
+    <command_interface name="position_pid">
+      <param name="min">0.0</param>
+      <param name="max">0.10</param>
+    </command_interface>
+    <state_interface name="position">
+      <param name="initial_value">0.0</param>
+    </state_interface>
+    <state_interface name="velocity"/>
+    <state_interface name="effort"/>
+  </joint>
   </ros2_control>
 </robot>

File: src/yektemak_description/urdf/yektemak_wheels.xacro (robot description, xacro)
@@ -2,9 +2,9 @@
 <robot xmlns:xacro="http://www.ros.org/wiki/xacro">
   <!-- Teker parametreleri -->
-  <xacro:property name="wheel_radius" value="0.18"/>
-  <xacro:property name="wheel_width" value="0.10"/>
-  <xacro:property name="wheel_mass" value="4.0"/>
+  <xacro:property name="wheel_radius" value="0.10"/>
+  <xacro:property name="wheel_width" value="0.05"/>
+  <xacro:property name="wheel_mass" value="2.0"/>
   <!-- Tekerlerin gövde üzerindeki konumları -->
-  <xacro:property name="wheel_x_position" value="0.42"/>
+  <xacro:property name="wheel_x_position" value="0.28"/>
   <xacro:property
     name="wheel_y_position"

Commit message: feat(description): add low front LiDAR and IMU, fix lift ros2_control
- 2D LiDAR on front bumper at 11 cm so it still sees with a pallet loaded
- IMU at body center
- Lift PID gains tuned for 6 kg platform + 55 kg loaded pallet
- Wheel joints exported as state interfaces (joint_states / TF)
- Base mass 80 kg, low wheel friction for planar_move stability
- use_sim xacro arg; display.launch.py uses use_sim:=false
- Remove ': ' and quotes from xacro comments (breaks gazebo_ros2_control YAML parsing)

File: src/yektemak_description/urdf/yektemak_base.xacro (robot description, xacro)
@@ -8,5 +8,5 @@
   <xacro:property name="base_ground_clearance" value="0.04"/>
   <!-- Yaklaşık gövde kütlesi -->
-  <xacro:property name="base_mass" value="35.0"/>
+  <xacro:property name="base_mass" value="80.0"/>
   <!-- Zemindeki referans noktası -->
   <link name="base_footprint"/>

File: src/yektemak_description/urdf/yektemak_gazebo.xacro (robot description, xacro)
@@ -1,56 +1,52 @@
+<?xml version="1.0"?>
 <robot xmlns:xacro="http://www.ros.org/wiki/xacro">
+  <!-- ================= Görünüm ve sürtünme ================= -->
   <gazebo reference="base_link">
     <material>Gazebo/Blue</material>
   </gazebo>
-  <gazebo reference="front_left_wheel_link">
-    <material>Gazebo/Black</material>
-    <mu1>1.0</mu1>
-    <mu2>1.0</mu2>
-    <kp>1000000.0</kp>
-    <kd>100.0</kd>
-  </gazebo>
-  <gazebo reference="front_right_wheel_link">
-    <material>Gazebo/Black</material>
-    <mu1>1.0</mu1>
-    <mu2>1.0</mu2>
-    <kp>1000000.0</kp>
-    <kd>100.0</kd>
-  </gazebo>
-  <gazebo reference="rear_left_wheel_link">
-    <material>Gazebo/Black</material>
-    <mu1>1.0</mu1>
-    <mu2>1.0</mu2>
-    <kp>1000000.0</kp>
-    <kd>100.0</kd>
-  </gazebo>
-  <gazebo reference="rear_right_wheel_link">
-    <material>Gazebo/Black</material>
-    <mu1>1.0</mu1>
-    <mu2>1.0</mu2>
-    <kp>1000000.0</kp>
-    <kd>100.0</kd>
-  </gazebo>
+  <!-- planar_move tum linklerin hizini her adimda kendisi ayarlar ve
+       tekerlerin donmesine izin vermez. Bu yuzden teker-zemin surtunmesi
+       dusuk tutulur; aksi halde tekerler fren yapar ve yuklu robot one/arkaya
+       devrilmeye calisir. Surus dinamigini planar_move belirler. -->
+  <xacro:macro name="wheel_gazebo" params="name">
+    <gazebo reference="${name}_wheel_link">
+      <material>Gazebo/DarkGrey</material>
+      <mu1>0.02</mu1>
+      <mu2>0.02</mu2>
+      <kp>1000000.0</kp>
+      <kd>100.0</kd>
+    </gazebo>
+  </xacro:macro>
+  <xacro:wheel_gazebo name="front_left"/>
+  <xacro:wheel_gazebo name="front_right"/>
+  <xacro:wheel_gazebo name="rear_left"/>
+  <xacro:wheel_gazebo name="rear_right"/>
+  <!-- Paleti kaydırmadan taşımak için yüksek sürtünmeli üst yüzey -->
   <gazebo reference="lift_platform_link">
     <material>Gazebo/Yellow</material>
-    <mu1>10.0</mu1>
-    <mu2>10.0</mu2>
-    <kp>1000000.0</kp>
-    <kd>100.0</kd>
-    <minDepth>0.001</minDepth>
-    <maxVel>0.01</maxVel>
+    <mu1>1.2</mu1>
+    <mu2>1.2</mu2>
   </gazebo>
   <gazebo reference="front_marker_link">
     <material>Gazebo/Red</material>
   </gazebo>
-    <gazebo>
-    <plugin
-      name="yektemak_planar_move"
-      filename="libgazebo_ros_planar_move.so">
+  <gazebo reference="lidar_link">
+    <material>Gazebo/FlatBlack</material>
+  </gazebo>
+  <gazebo reference="lidar_bracket_link">
+    <material>Gazebo/Grey</material>
+  </gazebo>
+  <!-- ================= Sürüş =================
+       planar_move gövdeyi doğrudan hız komutuyla sürer; 4 tekerli skid-steer
+       temasından çok daha kararlıdır. Navigasyon tarafında vy = 0 tutulur,
+       yani robot diferansiyel sürüşlü gibi davranır (gerçek araca uygun).
+  -->
+  <gazebo>
+    <plugin name="yektemak_planar_move" filename="libgazebo_ros_planar_move.so">
       <ros>
         <namespace>/</namespace>
-        <remapping>cmd_vel:=cmd_vel</remapping>
-        <remapping>odom:=odom</remapping>
       </ros>
-      <update_rate>100.0</update_rate>
+      <!-- Her fizik adiminda (1 kHz) hiz uygulanir; yukluyken devrilmeyi onler -->
+      <update_rate>1000.0</update_rate>
       <publish_rate>50.0</publish_rate>
       <publish_odom>true</publish_odom>
@@ -58,17 +54,110 @@
       <odometry_frame>odom</odometry_frame>
       <robot_base_frame>base_footprint</robot_base_frame>
+      <covariance_x>0.0001</covariance_x>
+      <covariance_y>0.0001</covariance_y>
+      <covariance_yaw>0.001</covariance_yaw>
     </plugin>
   </gazebo>
-    <!-- Kaldırma platformu için ROS 2 Control -->
+  <!-- ================= Lift - ros2_control ================= -->
   <gazebo>
-    <plugin
-      name="gazebo_ros2_control"
-      filename="libgazebo_ros2_control.so">
+    <plugin name="gazebo_ros2_control" filename="libgazebo_ros2_control.so">
       <robot_param>robot_description</robot_param>
       <robot_param_node>robot_state_publisher</robot_param_node>
-      <parameters>
-        $(find yektemak_gazebo)/config/controllers.yaml
-      </parameters>
+      <parameters>$(find yektemak_description)/config/ros2_controllers.yaml</parameters>
     </plugin>
   </gazebo>
+  <!-- ================= Palet baglayici =================
+       Lift kalkinca /pallet_attacher/attach (data true) ile ustteki palet
+       robota kilitlenir, indirince (data false) birakilir.
+       Kaynak - yektemak_gazebo_plugins paketi -->
+  <gazebo>
+    <plugin name="pallet_attacher" filename="libyektemak_pallet_attacher.so">
+      <ros>
+        <namespace>/</namespace>
+      </ros>
+      <parent_link>lift_platform_link</parent_link>
+      <target_prefix>pallet</target_prefix>
+      <max_xy_distance>0.25</max_xy_distance>
+      <max_yaw_error>0.35</max_yaw_error>
+    </plugin>
+  </gazebo>
+  <!-- ================= 2D LiDAR =================
+       Ön tamponda, +-100 derece görüş. Daha geniş açı gövdeye/tekerlere çarpar.
+  -->
+  <gazebo reference="lidar_link">
+    <sensor name="front_lidar" type="ray">
+      <always_on>true</always_on>
+      <visualize>false</visualize>
+      <update_rate>10.0</update_rate>
+      <pose>0 0 0 0 0 0</pose>
+      <ray>
+        <scan>
+          <horizontal>
+            <samples>401</samples>
+            <resolution>1</resolution>
+            <min_angle>-1.745329</min_angle>
+            <max_angle>1.745329</max_angle>
+          </horizontal>
+        </scan>
+        <range>
+          <min>0.10</min>
+          <max>20.0</max>
+          <resolution>0.01</resolution>
+        </range>
+        <noise>
+          <type>gaussian</type>
+          <mean>0.0</mean>
+          <stddev>0.005</stddev>
+        </noise>
+      </ray>
+      <plugin name="front_lidar_plugin" filename="libgazebo_ros_ray_sensor.so">
+        <ros>
+          <namespace>/</namespace>
+          <remapping>~/out:=scan_raw</remapping>
+        </ros>
+        <output_type>sensor_msgs/LaserScan</output_type>
+        <frame_name>lidar_link</frame_name>
+      </plugin>
+    </sensor>
+  </gazebo>
+  <!-- ================= IMU ================= -->
+  <gazebo reference="imu_link">
+    <sensor name="imu_sensor" type="imu">
+      <always_on>true</always_on>
+      <update_rate>100.0</update_rate>
+      <visualize>false</visualize>
+      <imu>
+        <angular_velocity>
+          <z>
+            <noise type="gaussian">
+              <mean>0.0</mean>
+              <stddev>0.0005</stddev>
+            </noise>
+          </z>
+        </angular_velocity>
+        <linear_acceleration>
+          <x>
+            <noise type="gaussian">
+              <mean>0.0</mean>
+              <stddev>0.01</stddev>
+            </noise>
+          </x>
+          <y>
+            <noise type="gaussian">
+              <mean>0.0</mean>
+              <stddev>0.01</stddev>
+            </noise>
+          </y>
+        </linear_acceleration>
+      </imu>
+      <plugin name="imu_plugin" filename="libgazebo_ros_imu_sensor.so">
+        <ros>
+          <namespace>/</namespace>
+          <remapping>~/out:=imu/data</remapping>
+        </ros>
+        <initial_orientation_as_reference>false</initial_orientation_as_reference>
+        <frame_name>imu_link</frame_name>
+      </plugin>
+    </sensor>
+  </gazebo>
 </robot>

File: src/yektemak_description/urdf/yektemak_robot.urdf.xacro (robot description, xacro)
@@ -1,19 +1,16 @@
 <?xml version="1.0"?>
-<robot
-  name="yektemak_robot"
-  xmlns:xacro="http://www.ros.org/wiki/xacro">
-  <!-- Renk tanımları -->
+<robot name="yektemak_robot" xmlns:xacro="http://www.ros.org/wiki/xacro">
+  <!-- Gazebo eklentilerini (sürüş, sensör, ros2_control) dahil et.
+       RVizde sadece modeli gormek icin use_sim argumanini false verin -->
+  <xacro:arg name="use_sim" default="true"/>
   <xacro:include filename="yektemak_materials.xacro"/>
-  <!-- Ana gövde -->
   <xacro:include filename="yektemak_base.xacro"/>
-  <!-- Dört teker -->
   <xacro:include filename="yektemak_wheels.xacro"/>
-  <!-- Palet kaldırma platformu -->
   <xacro:include filename="yektemak_lift.xacro"/>
-  <!-- Ön yön işareti -->
   <xacro:include filename="yektemak_markers.xacro"/>
-  <!-- Kaldırma sistemi ROS 2 Control arayüzü -->
-  <xacro:include filename="yektemak_ros2_control.xacro"/>
-  <!-- Gazebo fizik ve görünüm ayarları -->
-  <xacro:include filename="yektemak_gazebo.xacro"/>
+  <xacro:include filename="yektemak_sensors.xacro"/>
+  <xacro:if value="$(arg use_sim)">
+    <xacro:include filename="yektemak_ros2_control.xacro"/>
+    <xacro:include filename="yektemak_gazebo.xacro"/>
+  </xacro:if>
 </robot>

File: src/yektemak_description/urdf/yektemak_ros2_control.xacro (robot description, xacro)
@@ -1,22 +1,44 @@
+<?xml version="1.0"?>
 <robot xmlns:xacro="http://www.ros.org/wiki/xacro">
+  <!--
+    Gazebo ros2_control arayüzü
+    - lift_platform_joint - position_pid komut arayüzü. Gazebo eklemi
+      kuvvetle (PID) sürer; yüklü palette gerçekçi davranır.
+      Not - position_pid dışarıya "position" adıyla açılır, bu yüzden
+      position_controllers/JointGroupPositionController ile çalışır.
+    - Tekerlekler - sadece durum arayüzü (joint_states / TF için).
+      Sürüşü gazebo_ros_planar_move yapar.
+  -->
   <ros2_control name="YektemakGazeboSystem" type="system">
     <hardware>
       <plugin>gazebo_ros2_control/GazeboSystem</plugin>
     </hardware>
-  <joint name="lift_platform_joint">
-    <param name="pos_kp">6000.0</param>
-    <param name="pos_ki">50.0</param>
-    <param name="pos_kd">150.0</param>
-    <param name="pos_max_integral_error">100.0</param>
-    <command_interface name="position_pid">
-      <param name="min">0.0</param>
-      <param name="max">0.10</param>
-    </command_interface>
-    <state_interface name="position">
-      <param name="initial_value">0.0</param>
-    </state_interface>
-    <state_interface name="velocity"/>
-    <state_interface name="effort"/>
-  </joint>
+    <joint name="lift_platform_joint">
+      <!-- gazebo_ros2_control pos_ onekli parametreleri PID kazanci olarak okur.
+           Kazanclar 6 kg platform + 55 kg yuklu palet icin ayarlandi
+           (dogal frekans ~26 rad/s, sonum orani ~0.65). -->
+      <param name="pos_kp">40000.0</param>
+      <param name="pos_ki">8000.0</param>
+      <param name="pos_kd">2000.0</param>
+      <param name="pos_max_integral_error">3000.0</param>
+      <command_interface name="position_pid">
+        <param name="min">0.0</param>
+        <param name="max">${lift_max_height}</param>
+      </command_interface>
+      <state_interface name="position">
+        <param name="initial_value">0.0</param>
+      </state_interface>
+      <state_interface name="velocity"/>
+    </joint>
+    <xacro:macro name="wheel_state_only" params="name">
+      <joint name="${name}_wheel_joint">
+        <state_interface name="position"/>
+        <state_interface name="velocity"/>
+      </joint>
+    </xacro:macro>
+    <xacro:wheel_state_only name="front_left"/>
+    <xacro:wheel_state_only name="front_right"/>
+    <xacro:wheel_state_only name="rear_left"/>
+    <xacro:wheel_state_only name="rear_right"/>
   </ros2_control>
 </robot>
