Commit message: feat(fleet): multi-robot factory simulation
- 36 x 24 m factory: inbound docks, storage, production line, shipping,
  chargers, office; generated by tools/generate_factory.py
- Robot description: ns / frame prefix / body color args; per-robot unique
  sensor and plugin names; absolute sensor topics (sensor plugins ignore
  the namespace of the second robot in Gazebo Classic)
- spawn_robot.launch.py, factory.launch.py, robot_navigation.launch.py
  (own Nav2 launch on a shared /tf tree with prefixed frames)
- Factory map (SLAM), fleet RViz config, fleet_sim.launch.py
- Lifecycle bond timeout 30 s for slow startups

File: src/yektemak_description/urdf/yektemak_gazebo.xacro (robot description, xacro)
@@ -3,5 +3,5 @@
   <!-- ================= Görünüm ve sürtünme ================= -->
   <gazebo reference="base_link">
-    <material>Gazebo/Blue</material>
+    <material>Gazebo/${body_color}</material>
   </gazebo>
   <!-- planar_move tum linklerin hizini her adimda kendisi ayarlar ve
@@ -43,7 +43,7 @@
   -->
   <gazebo>
-    <plugin name="yektemak_planar_move" filename="libgazebo_ros_planar_move.so">
+    <plugin name="${ns}planar_move" filename="libgazebo_ros_planar_move.so">
       <ros>
-        <namespace>/</namespace>
+        <namespace>/${ns}</namespace>
       </ros>
       <!-- Her fizik adiminda (1 kHz) hiz uygulanir; yukluyken devrilmeyi onler -->
@@ -52,6 +52,6 @@
       <publish_odom>true</publish_odom>
       <publish_odom_tf>true</publish_odom_tf>
-      <odometry_frame>odom</odometry_frame>
-      <robot_base_frame>base_footprint</robot_base_frame>
+      <odometry_frame>${prefix}odom</odometry_frame>
+      <robot_base_frame>${prefix}base_footprint</robot_base_frame>
       <covariance_x>0.0001</covariance_x>
       <covariance_y>0.0001</covariance_y>
@@ -62,4 +62,7 @@
   <gazebo>
     <plugin name="gazebo_ros2_control" filename="libgazebo_ros2_control.so">
+      <ros>
+        <namespace>/${ns}</namespace>
+      </ros>
       <robot_param>robot_description</robot_param>
       <robot_param_node>robot_state_publisher</robot_param_node>
@@ -72,7 +75,7 @@
        Kaynak - yektemak_gazebo_plugins paketi -->
   <gazebo>
-    <plugin name="pallet_attacher" filename="libyektemak_pallet_attacher.so">
+    <plugin name="${ns}pallet_attacher" filename="libyektemak_pallet_attacher.so">
       <ros>
-        <namespace>/</namespace>
+        <namespace>/${ns}</namespace>
       </ros>
       <parent_link>lift_platform_link</parent_link>
@@ -82,9 +85,12 @@
     </plugin>
   </gazebo>
+  <!-- Not - sensor ve eklenti adlari ns ile baslar. Iki robotta ayni ad
+       kullanilirsa Gazebo eklentileri karisiyor ve bir robotun LiDAR verisi
+       digerinin topicine akiyor. -->
   <!-- ================= 2D LiDAR =================
        Ön tamponda, +-100 derece görüş. Daha geniş açı gövdeye/tekerlere çarpar.
   -->
   <gazebo reference="lidar_link">
-    <sensor name="front_lidar" type="ray">
+    <sensor name="${ns}front_lidar" type="ray">
       <always_on>true</always_on>
       <visualize>false</visualize>
@@ -111,11 +117,13 @@
         </noise>
       </ray>
-      <plugin name="front_lidar_plugin" filename="libgazebo_ros_ray_sensor.so">
+      <plugin name="${ns}front_lidar_plugin" filename="libgazebo_ros_ray_sensor.so">
         <ros>
-          <namespace>/</namespace>
-          <remapping>~/out:=scan_raw</remapping>
+          <!-- Sensor eklentilerinde namespace guvenilir degil (coklu robotta
+               ikinci robotun sensoru ilk robotun namespace inde aciliyor).
+               Bu yuzden topic mutlak adla verilir. -->
+          <remapping>~/out:=${'/' + ns if ns else ''}/scan_raw</remapping>
         </ros>
         <output_type>sensor_msgs/LaserScan</output_type>
-        <frame_name>lidar_link</frame_name>
+        <frame_name>${prefix}lidar_link</frame_name>
       </plugin>
     </sensor>
@@ -123,5 +131,5 @@
   <!-- ================= IMU ================= -->
   <gazebo reference="imu_link">
-    <sensor name="imu_sensor" type="imu">
+    <sensor name="${ns}imu_sensor" type="imu">
       <always_on>true</always_on>
       <update_rate>100.0</update_rate>
@@ -151,11 +159,10 @@
         </linear_acceleration>
       </imu>
-      <plugin name="imu_plugin" filename="libgazebo_ros_imu_sensor.so">
+      <plugin name="${ns}imu_plugin" filename="libgazebo_ros_imu_sensor.so">
         <ros>
-          <namespace>/</namespace>
-          <remapping>~/out:=imu/data</remapping>
+          <remapping>~/out:=${'/' + ns if ns else ''}/imu/data</remapping>
         </ros>
         <initial_orientation_as_reference>false</initial_orientation_as_reference>
-        <frame_name>imu_link</frame_name>
+        <frame_name>${prefix}imu_link</frame_name>
       </plugin>
     </sensor>

File: src/yektemak_description/urdf/yektemak_robot.urdf.xacro (robot description, xacro)
@@ -4,4 +4,14 @@
        RVizde sadece modeli gormek icin use_sim argumanini false verin -->
   <xacro:arg name="use_sim" default="true"/>
+  <!-- Coklu robot icin namespace (ornek robot1). Bos = tek robot.
+       Gazebo eklentileri bu namespace altinda yayin yapar, frame adlari
+       ns/ oneki alir (robot1/odom, robot1/base_footprint). Link adlari ayni
+       kalir; robot_state_publisher frame_prefix ile oneki ekler. -->
+  <xacro:arg name="ns" default=""/>
+  <xacro:property name="ns" value="$(arg ns)"/>
+  <xacro:property name="prefix" value="${ns + '/' if ns else ''}"/>
+  <!-- Gazebo govde rengi (Gazebo/Blue, Gazebo/Orange ...) -->
+  <xacro:arg name="body_color" default="Blue"/>
+  <xacro:property name="body_color" value="$(arg body_color)"/>
   <xacro:include filename="yektemak_materials.xacro"/>
   <xacro:include filename="yektemak_base.xacro"/>

Commit message: feat: rear LiDAR, 18 cm lift, fleet traffic priority, stale Gazebo guard
- Rear 2D LiDAR (mirror of the front one) as a second costmap source,
  own laser filter (/scan_rear_raw -> /scan_rear)
- Lift stroke 0.10 -> 0.18 m: carried pallet rises 14 cm so its runners
  clear the 11 cm LiDAR plane and the robot sees all around while loaded
- Fleet traffic: when two busy robots come within 2.4 m the lower priority
  one (unloaded / newer task) yields until 3.2 m apart; 25 s max hold with
  cooldown against deadlock; agent pauses only Nav2, never docking/lift
- Launch refuses to start if an old gzserver is running (robots would be
  spawned into the old world); fleet manager verifies the factory world
  and warns on the dashboard
- Dashboard: 'Yol veriyor' badge and hold ring

File: src/yektemak_description/urdf/yektemak_gazebo.xacro (robot description, xacro)
@@ -33,4 +33,10 @@
   <gazebo reference="lidar_link">
     <material>Gazebo/FlatBlack</material>
+  </gazebo>
+  <gazebo reference="rear_lidar_link">
+    <material>Gazebo/FlatBlack</material>
+  </gazebo>
+  <gazebo reference="rear_lidar_bracket_link">
+    <material>Gazebo/Grey</material>
   </gazebo>
   <gazebo reference="lidar_bracket_link">
@@ -133,4 +139,40 @@
     </sensor>
   </gazebo>
+  <!-- ================= Arka 2D LiDAR ================= -->
+  <gazebo reference="rear_lidar_link">
+    <sensor name="${ns}rear_lidar" type="ray">
+      <always_on>true</always_on>
+      <visualize>false</visualize>
+      <update_rate>10.0</update_rate>
+      <pose>0 0 0 0 0 0</pose>
+      <ray>
+        <scan>
+          <horizontal>
+            <samples>401</samples>
+            <resolution>1</resolution>
+            <min_angle>-1.745329</min_angle>
+            <max_angle>1.745329</max_angle>
+          </horizontal>
+        </scan>
+        <range>
+          <min>0.10</min>
+          <max>20.0</max>
+          <resolution>0.01</resolution>
+        </range>
+        <noise>
+          <type>gaussian</type>
+          <mean>0.0</mean>
+          <stddev>0.005</stddev>
+        </noise>
+      </ray>
+      <plugin name="${ns}rear_lidar_plugin" filename="libgazebo_ros_ray_sensor.so">
+        <ros>
+          <remapping>~/out:=${'/' + ns if ns else ''}/scan_rear_raw</remapping>
+        </ros>
+        <output_type>sensor_msgs/LaserScan</output_type>
+        <frame_name>${prefix}rear_lidar_link</frame_name>
+      </plugin>
+    </sensor>
+  </gazebo>
   <!-- ================= IMU ================= -->
   <gazebo reference="imu_link">

File: src/yektemak_description/urdf/yektemak_lift.xacro (robot description, xacro)
@@ -7,5 +7,5 @@
   <xacro:property name="lift_platform_mass" value="6.0"/>
   <xacro:property name="lift_platform_clearance" value="0.01"/>
-  <xacro:property name="lift_max_height" value="0.10"/>
+  <xacro:property name="lift_max_height" value="0.18"/>
   <!-- Paleti kaldıracak üst platform -->
   <link name="lift_platform_link">

File: src/yektemak_description/urdf/yektemak_sensors.xacro (robot description, xacro)
@@ -61,4 +61,53 @@
       rpy="0 0 0"/>
   </joint>
+  <!-- Arka 2D LiDAR - on LiDARin simetrigi, geriye bakar. Geri giderken ve
+       robotlar karsilastiginda arkayi da gormek icin. Costmapte ikinci
+       gozlem kaynagi olarak kullanilir. -->
+  <link name="rear_lidar_bracket_link">
+    <visual>
+      <origin xyz="0 0 0" rpy="0 0 0"/>
+      <geometry>
+        <box size="0.07 0.08 0.02"/>
+      </geometry>
+      <material name="yektemak_gray"/>
+    </visual>
+  </link>
+  <joint name="rear_lidar_bracket_joint" type="fixed">
+    <parent link="base_link"/>
+    <child link="rear_lidar_bracket_link"/>
+    <origin
+      xyz="${-(base_length / 2.0 + 0.035)} 0
+           ${lidar_height_from_ground - lidar_length / 2.0 - 0.01
+             - (base_ground_clearance + base_height / 2.0)}"
+      rpy="0 0 0"/>
+  </joint>
+  <link name="rear_lidar_link">
+    <visual>
+      <origin xyz="0 0 0" rpy="0 0 0"/>
+      <geometry>
+        <cylinder radius="${lidar_radius}" length="${lidar_length}"/>
+      </geometry>
+      <material name="yektemak_dark"/>
+    </visual>
+    <collision>
+      <origin xyz="0 0 0" rpy="0 0 0"/>
+      <geometry>
+        <cylinder radius="${lidar_radius}" length="${lidar_length}"/>
+      </geometry>
+    </collision>
+    <inertial>
+      <origin xyz="0 0 0" rpy="0 0 0"/>
+      <mass value="0.3"/>
+      <inertia ixx="0.0002" ixy="0" ixz="0" iyy="0.0002" iyz="0" izz="0.0002"/>
+    </inertial>
+  </link>
+  <joint name="rear_lidar_joint" type="fixed">
+    <parent link="base_link"/>
+    <child link="rear_lidar_link"/>
+    <origin
+      xyz="${-lidar_x} 0
+           ${lidar_height_from_ground - (base_ground_clearance + base_height / 2.0)}"
+      rpy="0 0 ${pi}"/>
+  </joint>
   <!-- IMU - gövde merkezinde -->
   <link name="imu_link">
